File: eagle/ESP32FishLightBoard.sch (EAGLE design)
At the start: 5 parts, among them J1 1X2-3.5MM, U1 SN74HCT04N

Commit message: added pull-down resistor to board
Parts:
- added R1: 4.7k, adafruit:FLIPFLOP-RES
Connections:
- net GND: now also R1.2
- net IO17: now also R1.1
Changed lines of the file:
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@@
 <part name="JPLED" library="jumper" library_urn="urn:adsk.eagle:library:252" deviceset="JP2E" device="" package3d_urn="urn:adsk.eagle:package:15452/1"/>
 <part name="U1" library="UltralibrarianImported" deviceset="SN74HCT04N" device=""/>
+<part name="R1" library="adafruit" library_urn="urn:adsk.eagle:library:420" deviceset="FLIPFLOP-RES" device="" package3d_urn="urn:adsk.eagle:package:6240726/1" value="4.7k"/>
 </parts>
 <sheets>
@@
 <attribute name="NAME" x="127.3556" y="62.4586" size="2.0828" layer="95" ratio="6" rot="SR0"/>
 <attribute name="VALUE" x="126.7206" y="59.9186" size="2.0828" layer="96" ratio="6" rot="SR0"/>
+</instance>
+<instance part="R1" gate="G$1" x="101.6" y="73.66" smashed="yes">
+<attribute name="NAME" x="97.79" y="75.1586" size="1.778" layer="95"/>
+<attribute name="VALUE" x="97.79" y="70.358" size="1.778" layer="96"/>
 </instance>
 </instances>
@@
 <label x="129.54" y="91.44" size="1.778" layer="95"/>
 </segment>
+<segment>
+<pinref part="R1" gate="G$1" pin="2"/>
+<wire x1="106.68" y1="73.66" x2="116.84" y2="73.66" width="0.1524" layer="91"/>
+<label x="114.3" y="73.66" size="1.778" layer="95" align="bottom-right"/>
+</segment>
 </net>
 <net name="N$1" class="1">
@@
 <label x="101.6" y="53.34" size="1.778" layer="95"/>
 </segment>
+<segment>
+<pinref part="R1" gate="G$1" pin="1"/>
+<wire x1="96.52" y1="73.66" x2="86.36" y2="73.66" width="0.1524" layer="91"/>
+<label x="88.9" y="73.66" size="1.778" layer="95"/>
+</segment>
 </net>
