File: eagle/projects/ESP32FishLightBoard.sch (EAGLE design)
At the start: 9 parts, among them U1 SN74HCT04N

Commit message: updated to v1.1 PCB
Parts:
- added BZR: F/QMX, buzzer:F/QMX
- added OLED: 22-27-2041-04, con-molex:22-27-2041-04
- added T3V3, TDAT, TGND: WIREPAD2,54/1,0, wirepad:WIREPAD2,54/1,0
Connections:
- new net 3V3: OLED-2.S, T3V3.P, U$1.3V3
- new net IO12: U$1.IO12
- new net IO14: U$1.IO14
- new net IO15: BZR.2, U$1.IO15
- new net IO16: TDAT.P, U$1.IO16
- new net SCL: OLED-3.S, U$1.IO22
- new net SDA: OLED-4.S, U$1.IO21
- net GND: now also BZR.1, OLED-1.S, TGND.P
Changed lines of the file:
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@@
 <part name="LDAT" library="wirepad" library_urn="urn:adsk.eagle:library:412" deviceset="WIREPAD" device="2,54/1,0" package3d_urn="urn:adsk.eagle:package:30828/1"/>
 <part name="LVCC" library="wirepad" library_urn="urn:adsk.eagle:library:412" deviceset="WIREPAD" device="2,54/1,0" package3d_urn="urn:adsk.eagle:package:30828/1"/>
+<part name="TGND" library="wirepad" library_urn="urn:adsk.eagle:library:412" deviceset="WIREPAD" device="2,54/1,0" package3d_urn="urn:adsk.eagle:package:30828/1"/>
+<part name="TDAT" library="wirepad" library_urn="urn:adsk.eagle:library:412" deviceset="WIREPAD" device="2,54/1,0" package3d_urn="urn:adsk.eagle:package:30828/1"/>
+<part name="T3V3" library="wirepad" library_urn="urn:adsk.eagle:library:412" deviceset="WIREPAD" device="2,54/1,0" package3d_urn="urn:adsk.eagle:package:30828/1"/>
+<part name="BZR" library="buzzer" library_urn="urn:adsk.eagle:library:113" deviceset="F/QMX" device="" package3d_urn="urn:adsk.eagle:package:5278/1"/>
+<part name="OLED" library="con-molex" library_urn="urn:adsk.eagle:library:165" deviceset="22-?-04" device="27-2041" package3d_urn="urn:adsk.eagle:package:8078649/1"/>
 </parts>
 <sheets>
@@
 <attribute name="NAME" x="34.417" y="98.3742" size="1.778" layer="95"/>
 </instance>
+<instance part="TGND" gate="G$1" x="0" y="91.44" smashed="yes">
+<attribute name="NAME" x="-1.143" y="93.2942" size="1.778" layer="95"/>
+</instance>
+<instance part="TDAT" gate="G$1" x="0" y="96.52" smashed="yes">
+<attribute name="NAME" x="-1.143" y="98.3742" size="1.778" layer="95"/>
+</instance>
+<instance part="T3V3" gate="G$1" x="0" y="101.6" smashed="yes">
+<attribute name="NAME" x="-1.143" y="103.4542" size="1.778" layer="95"/>
+</instance>
+<instance part="BZR" gate="G$1" x="-5.08" y="63.5" smashed="yes">
+<attribute name="NAME" x="-7.62" y="69.85" size="1.778" layer="95"/>
+</instance>
+<instance part="OLED" gate="-1" x="96.52" y="111.76" smashed="yes">
+<attribute name="NAME" x="99.06" y="110.998" size="1.524" layer="95"/>
+</instance>
+<instance part="OLED" gate="-2" x="96.52" y="106.68" smashed="yes">
+<attribute name="NAME" x="99.06" y="105.918" size="1.524" layer="95"/>
+</instance>
+<instance part="OLED" gate="-3" x="96.52" y="101.6" smashed="yes">
+<attribute name="NAME" x="99.06" y="100.838" size="1.524" layer="95"/>
+</instance>
+<instance part="OLED" gate="-4" x="96.52" y="96.52" smashed="yes">
+<attribute name="NAME" x="99.06" y="95.758" size="1.524" layer="95"/>
+</instance>
 </instances>
 <busses>
@@
 <wire x1="33.02" y1="40.64" x2="22.86" y2="40.64" width="0.1524" layer="91"/>
 <label x="25.4" y="40.64" size="1.778" layer="95"/>
+</segment>
+<segment>
+<pinref part="BZR" gate="G$1" pin="1"/>
+<wire x1="-7.62" y1="60.96" x2="-17.78" y2="60.96" width="0.1524" layer="91"/>
+<label x="-15.24" y="60.96" size="1.778" layer="95"/>
+</segment>
+<segment>
+<pinref part="TGND" gate="G$1" pin="P"/>
+<wire x1="2.54" y1="91.44" x2="12.7" y2="91.44" width="0.1524" layer="91"/>
+<label x="10.16" y="91.44" size="1.778" layer="95" align="bottom-right"/>
+</segment>
+<segment>
+<pinref part="OLED" gate="-1" pin="S"/>
+<wire x1="93.98" y1="111.76" x2="86.36" y2="111.76" width="0.1524" layer="91"/>
+<label x="88.9" y="111.76" size="1.778" layer="95"/>
 </segment>
 </net>
@@
 </segment>
 </net>
+<net name="IO12" class="0">
+<segment>
+<pinref part="U$1" gate="G$1" pin="IO12"/>
+<wire x1="68.58" y1="55.88" x2="78.74" y2="55.88" width="0.1524" layer="91"/>
+<label x="76.2" y="55.88" size="1.778" layer="95" align="bottom-right"/>
+</segment>
+</net>
+<net name="IO14" class="0">
+<segment>
+<pinref part="U$1" gate="G$1" pin="IO14"/>
+<wire x1="68.58" y1="53.34" x2="78.74" y2="53.34" width="0.1524" layer="91"/>
+<label x="76.2" y="53.34" size="1.778" layer="95" align="bottom-right"/>
+</segment>
+</net>
+<net name="IO16" class="0">
+<segment>
+<pinref part="U$1" gate="G$1" pin="IO16"/>
+<wire x1="33.02" y1="53.34" x2="22.86" y2="53.34" width="0.1524" layer="91"/>
+<label x="25.4" y="53.34" size="1.778" layer="95"/>
+</segment>
+<segment>
+<pinref part="TDAT" gate="G$1" pin="P"/>
+<wire x1="2.54" y1="96.52" x2="12.7" y2="96.52" width="0.1524" layer="91"/>
+<label x="10.16" y="96.52" size="1.778" layer="95" align="bottom-right"/>
+</segment>
+</net>
+<net name="3V3" class="0">
+<segment>
+<pinref part="T3V3" gate="G$1" pin="P"/>
+<wire x1="2.54" y1="101.6" x2="12.7" y2="101.6" width="0.1524" layer="91"/>
+<label x="10.16" y="101.6" size="1.778" layer="95" align="bottom-right"/>
+</segment>
+<segment>
+<pinref part="U$1" gate="G$1" pin="3V3"/>
+<wire x1="68.58" y1="25.4" x2="78.74" y2="25.4" width="0.1524" layer="91"/>
+<label x="76.2" y="25.4" size="1.778" layer="95" align="bottom-right"/>
+</segment>
+<segment>
+<pinref part="OLED" gate="-2" pin="S"/>
+<wire x1="93.98" y1="106.68" x2="86.36" y2="106.68" width="0.1524" layer="91"/>
+<label x="88.9" y="106.68" size="1.778" layer="95"/>
+</segment>
+</net>
+<net name="IO15" class="0">
+<segment>
+<pinref part="U$1" gate="G$1" pin="IO15"/>
+<wire x1="33.02" y1="63.5" x2="22.86" y2="63.5" width="0.1524" layer="91"/>
+<label x="25.4" y="63.5" size="1.778" layer="95"/>
+</segment>
+<segment>
+<pinref part="BZR" gate="G$1" pin="2"/>
+<wire x1="0" y1="60.96" x2="10.16" y2="60.96" width="0.1524" layer="91"/>
+<label x="7.62" y="60.96" size="1.778" layer="95" align="bottom-right"/>
+</segment>
+</net>
+<net name="SDA" class="0">
+<segment>
+<pinref part="OLED" gate="-4" pin="S"/>
+<wire x1="93.98" y1="96.52" x2="86.36" y2="96.52" width="0.1524" layer="91"/>
+<label x="88.9" y="96.52" size="1.778" layer="95"/>
+</segment>
+<segment>
+<pinref part="U$1" gate="G$1" pin="IO21"/>
+<wire x1="33.02" y1="38.1" x2="22.86" y2="38.1" width="0.1524" layer="91"/>
+<label x="25.4" y="38.1" size="1.778" layer="95"/>
+</segment>
+</net>
+<net name="SCL" class="0">
+<segment>
+<pinref part="OLED" gate="-3" pin="S"/>
+<wire x1="93.98" y1="101.6" x2="86.36" y2="101.6" width="0.1524" layer="91"/>
+<label x="88.9" y="101.6" size="1.778" layer="95"/>
+</segment>
+<segment>
+<pinref part="U$1" gate="G$1" pin="IO22"/>
+<wire x1="33.02" y1="30.48" x2="22.86" y2="30.48" width="0.1524" layer="91"/>
+<label x="25.4" y="30.48" size="1.778" layer="95"/>
+</segment>
+</net>

Commit message: Adding eagle for v1.1 board
Parts:
- added R2: 4.7k, adafruit:FLIPFLOP-RES
Connections:
- net 3V3: now also R2.2
- net IO16: now also R2.1
Changed lines of the file:
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@@
 <part name="BZR" library="buzzer" library_urn="urn:adsk.eagle:library:113" deviceset="F/QMX" device="" package3d_urn="urn:adsk.eagle:package:5278/1"/>
 <part name="OLED" library="con-molex" library_urn="urn:adsk.eagle:library:165" deviceset="22-?-04" device="27-2041" package3d_urn="urn:adsk.eagle:package:8078649/1"/>
+<part name="R2" library="adafruit" library_urn="urn:adsk.eagle:library:420" deviceset="FLIPFLOP-RES" device="" package3d_urn="urn:adsk.eagle:package:6240726/1" value="4.7k"/>
 </parts>
 <sheets>
@@
 <attribute name="NAME" x="99.06" y="95.758" size="1.524" layer="95"/>
 </instance>
+<instance part="R2" gate="G$1" x="99.06" y="22.86" smashed="yes">
+<attribute name="NAME" x="95.25" y="24.3586" size="1.778" layer="95"/>
+<attribute name="VALUE" x="95.25" y="19.558" size="1.778" layer="96"/>
+</instance>
 </instances>
 <busses>
@@
 <label x="10.16" y="96.52" size="1.778" layer="95" align="bottom-right"/>
 </segment>
+<segment>
+<pinref part="R2" gate="G$1" pin="1"/>
+<wire x1="93.98" y1="22.86" x2="88.9" y2="22.86" width="0.1524" layer="91"/>
+<label x="88.9" y="22.86" size="1.778" layer="95"/>
+</segment>
 </net>
 <net name="3V3" class="0">
@@
 <label x="88.9" y="106.68" size="1.778" layer="95"/>
 </segment>
-</net>
+<segment>
+<pinref part="R2" gate="G$1" pin="2"/>
+<wire x1="104.14" y1="22.86" x2="109.22" y2="22.86" width="0.1524" layer="91"/>
+<label x="109.22" y="22.86" size="1.778" layer="95"/>
+</segment>
+</net>
